Commit message: Jordan's Updates

File: src/41068_ignition_bringup_v1/41068_ignition_bringup/urdf_husky/husky.gazebo.xacro (robot description, xacro)
@@ -6,4 +6,21 @@
   <xacro:arg name="gz_model_name" default="husky"/>
   <xacro:property name="gz_model_name" value="$(arg gz_model_name)"/>
+  <!-- Sensor performance knobs.
+       Ignition renders every camera and lidar on a single sensor thread, so an
+       expensive camera directly throttles the lidar. On software-GL machines
+       (WSL) a 720x480 RGBD camera starves the lidar to well below 1 Hz, which
+       breaks SLAM and the Nav2 costmaps. These arguments let the launch trade
+       camera fidelity for the scan rate that navigation depends on. -->
+  <xacro:arg name="enable_camera"      default="false"/>
+  <xacro:arg name="lidar_update_rate"  default="10"/>
+  <xacro:arg name="lidar_samples"      default="360"/>
+  <xacro:arg name="camera_update_rate" default="3"/>
+  <xacro:arg name="camera_width"       default="720"/>
+  <xacro:arg name="camera_height"      default="480"/>
+  <xacro:property name="enable_camera" value="$(arg enable_camera)"/>
+  <!-- Which Gazebo system drives the base. See the plugin block below. -->
+  <xacro:arg name="drive_plugin" default="diff_drive"/>
+  <xacro:property name="drive_plugin" value="$(arg drive_plugin)"/>
+  <xacro:arg name="effective_wheel_separation" default="0.94"/>
   <xacro:include filename="$(find 41068_ignition_bringup)/urdf_husky/wheel.urdf.xacro"/>
   <gazebo reference="${prefix}imu_link">
@@ -75,13 +92,53 @@
     <material>Gazebo/Grey</material>
   </gazebo>
-  <!-- Move base directly without faffing around with diff drive controllers -->
-  <gazebo>
-    <plugin
-      filename="ignition-gazebo-velocity-control-system"
-      name="ignition::gazebo::systems::VelocityControl">
-      <topic>model/${gz_model_name}/cmd_vel</topic>
-    </plugin>
-  </gazebo>
-  <!-- Publish odometry separately -->
+  <!-- Drive the base.
+       DiffDrive commands the four wheel joints, so a turn is produced the way a
+       real skid-steer Husky produces one. The alternative, VelocityControl,
+       hard-sets the velocity of base_link only; measured on this repository it
+       tracks linear commands exactly but achieves just 0.045 rad/s of the
+       0.5 rad/s commanded yaw, because the wheel contacts resist a rotation
+       that no wheel is turning to create. Nav2 needs rotate-in-place for
+       RotateToGoal and for its spin recovery, so DiffDrive is the default.
+       Set drive_plugin:=velocity_control to compare. -->
+  <xacro:if value="${drive_plugin == 'diff_drive'}">
+    <gazebo>
+      <plugin
+        filename="ignition-gazebo-diff-drive-system"
+        name="ignition::gazebo::systems::DiffDrive">
+        <left_joint>${prefix}front_left_wheel_joint</left_joint>
+        <left_joint>${prefix}rear_left_wheel_joint</left_joint>
+        <right_joint>${prefix}front_right_wheel_joint</right_joint>
+        <right_joint>${prefix}rear_right_wheel_joint</right_joint>
+        <!-- A skid-steer's effective track is wider than its geometric track,
+             because turning drags the tyres sideways. Calibrated against the
+             measured yaw rate in test/movement_test.py; the geometric value is
+             the starting point. -->
+        <wheel_separation>$(arg effective_wheel_separation)</wheel_separation>
+        <wheel_radius>${wheel_radius}</wheel_radius>
+        <topic>model/${gz_model_name}/cmd_vel</topic>
+        <!-- DiffDrive also offers odometry, but this model keeps
+             OdometryPublisher (below) as the single odometry source. Point
+             DiffDrive's own output at unused topics so the two plugins never
+             publish to the same place. -->
+        <odom_topic>model/${gz_model_name}/diff_drive/odometry</odom_topic>
+        <tf_topic>model/${gz_model_name}/diff_drive/tf</tf_topic>
+        <frame_id>${prefix}odom</frame_id>
+        <child_frame_id>${prefix}base_link</child_frame_id>
+        <odom_publish_frequency>1</odom_publish_frequency>
+      </plugin>
+    </gazebo>
+  </xacro:if>
+  <xacro:if value="${drive_plugin == 'velocity_control'}">
+    <gazebo>
+      <plugin
+        filename="ignition-gazebo-velocity-control-system"
+        name="ignition::gazebo::systems::VelocityControl">
+        <topic>model/${gz_model_name}/cmd_vel</topic>
+      </plugin>
+    </gazebo>
+  </xacro:if>
+  <!-- Odometry. Differentiates the simulated pose rather than integrating wheel
+       encoders, so it does not accumulate the slip error that skid-steering
+       creates. The EKF fuses it with the IMU to publish odom->base_link. -->
   <gazebo>
     <plugin
@@ -107,10 +164,10 @@
       <visualize>$(arg laser_visual)</visualize>
       <topic>model/${gz_model_name}/scan</topic>
-      <update_rate>3</update_rate>
+      <update_rate>$(arg lidar_update_rate)</update_rate>
       <gz_frame_id>${prefix}base_scan</gz_frame_id>
       <ray>
         <scan>
           <horizontal>
-            <samples>360</samples>
+            <samples>$(arg lidar_samples)</samples>
             <resolution>1</resolution>
             <min_angle>0.0</min_angle>
@@ -132,4 +189,5 @@
     </sensor>
   </gazebo>
+  <xacro:if value="${enable_camera}">
   <gazebo reference="${prefix}camera_link">
     <sensor name="rgbd_camera" type="rgbd_camera">
@@ -137,6 +195,6 @@
         <horizontal_fov>2.0944</horizontal_fov>
         <image>
-          <width>720</width>
-          <height>480</height>
+          <width>$(arg camera_width)</width>
+          <height>$(arg camera_height)</height>
         </image>
         <clip>
@@ -159,5 +217,5 @@
       </camera>
       <always_on>1</always_on>
-      <update_rate>3</update_rate> <!--10-->
+      <update_rate>$(arg camera_update_rate)</update_rate>
       <visualize>$(arg camera_visual)</visualize>
       <topic>/model/${gz_model_name}/camera</topic>
@@ -165,3 +223,4 @@
     </sensor>
   </gazebo>
+  </xacro:if>
 </robot>

Commit message: Laptop

File: src/41068_ignition_bringup_v1/41068_ignition_bringup/urdf_husky/husky.gazebo.xacro (robot description, xacro)
@@ -73,5 +73,4 @@
       </plugin>
     </sensor>
-    <material>Gazebo/Grey</material>
   </gazebo>
   <!-- Move base directly without faffing around with diff drive controllers -->
@@ -102,5 +101,4 @@
   </gazebo>
   <gazebo reference="${prefix}base_scan">
-    <material>Gazebo/FlatBlack</material>
     <sensor type="gpu_lidar" name="lidar">
       <pose relative_to='${prefix}base_scan'>0 0 0 0 0 0</pose>

File: src/41068_ignition_bringup_v1/41068_ignition_bringup/urdf_husky/husky.urdf.xacro (robot description, xacro)
@@ -37,4 +37,5 @@
         <mesh filename="file://$(find 41068_ignition_bringup)/urdf_husky/meshes/top_chassis.dae"/>
       </geometry>
+      <material name="orange"/>
     </visual>
     <visual name="base_link_fixed_joint_lump__top_plate_link_visual_6">

File: src/41068_ignition_bringup_v1/41068_ignition_bringup/urdf_husky/wheel.urdf.xacro (robot description, xacro)
@@ -11,4 +11,5 @@
           <mesh filename="file://$(find 41068_ignition_bringup)/urdf_husky/meshes/wheel.dae"/>
         </geometry>
+        <material name="dark"/>
       </visual>
       <collision>
