Commit message: merge artifacts removed

File: install/41068_ignition_bringup/share/41068_ignition_bringup/urdf_husky/common_properties.urdf.xacro (robot description, xacro)
@@ -1 +1,34 @@
-/home/jordan/G25_RS1/RS1-Gr25/src/41068_ignition_bringup_v1/41068_ignition_bringup/urdf_husky/common_properties.urdf.xacro
+<?xml version="1.0" ?>
+<robot name="xacro_properties" xmlns:xacro="http://ros.org/wiki/xacro">
+  <!-- Init colour -->
+  <material name="black">
+      <color rgba="0.0 0.0 0.0 1.0"/>
+  </material>
+  <material name="dark">
+    <color rgba="0.3 0.3 0.3 1.0"/>
+  </material>
+  <material name="light_black">
+    <color rgba="0.4 0.4 0.4 1.0"/>
+  </material>
+  <material name="blue">
+    <color rgba="0.0 0.0 0.8 1.0"/>
+  </material>
+  <material name="green">
+    <color rgba="0.0 0.8 0.0 1.0"/>
+  </material>
+  <material name="grey">
+    <color rgba="0.5 0.5 0.5 1.0"/>
+  </material>
+  <material name="orange">
+    <color rgba="${255/255} ${108/255} ${10/255} 1.0"/>
+  </material>
+  <material name="brown">
+    <color rgba="${222/255} ${207/255} ${195/255} 1.0"/>
+  </material>
+  <material name="red">
+    <color rgba="0.8 0.0 0.0 1.0"/>
+  </material>
+  <material name="white">
+    <color rgba="1.0 1.0 1.0 1.0"/>
+  </material>
+</robot>

File: install/41068_ignition_bringup/share/41068_ignition_bringup/urdf_husky/husky.gazebo.xacro (robot description, xacro)
@@ -1 +1,255 @@
-/home/jordan/G25_RS1/RS1-Gr25/src/41068_ignition_bringup_v1/41068_ignition_bringup/urdf_husky/husky.gazebo.xacro
+<?xml version="1.0"?>
+<robot name="husky" xmlns:xacro="http://ros.org/wiki/xacro">
+  <xacro:arg name="laser_visual"  default="false" />
+  <xacro:arg name="camera_visual" default="false"/>
+  <xacro:arg name="imu_visual"    default="false"/>
+  <xacro:arg name="gz_model_name" default="husky"/>
+  <xacro:property name="gz_model_name" value="$(arg gz_model_name)"/>
+  <!-- Sensor performance knobs.
+       Ignition renders every camera and lidar on a single sensor thread, so an
+       expensive camera directly throttles the lidar. On software-GL machines
+       (WSL) a 720x480 RGBD camera starves the lidar to well below 1 Hz, which
+       breaks SLAM and the Nav2 costmaps. These arguments let the launch trade
+       camera fidelity for the scan rate that navigation depends on. -->
+  <xacro:arg name="enable_camera"      default="false"/>
+  <xacro:arg name="lidar_update_rate"  default="10"/>
+  <xacro:arg name="lidar_samples"      default="360"/>
+  <xacro:arg name="camera_update_rate" default="3"/>
+  <xacro:arg name="camera_width"       default="720"/>
+  <xacro:arg name="camera_height"      default="480"/>
+  <xacro:property name="enable_camera" value="$(arg enable_camera)"/>
+  <!-- Which Gazebo system drives the base. See the plugin block below. -->
+  <xacro:arg name="drive_plugin" default="diff_drive"/>
+  <xacro:property name="drive_plugin" value="$(arg drive_plugin)"/>
+  <xacro:arg name="effective_wheel_separation" default="0.94"/>
+  <xacro:include filename="$(find 41068_ignition_bringup)/urdf_husky/wheel.urdf.xacro"/>
+  <gazebo reference="${prefix}imu_link">
+    <sensor type="imu" name="imu">
+      <always_on>true</always_on>
+      <visualize>$(arg imu_visual)</visualize>
+      <update_rate>100</update_rate>
+      <topic>model/${gz_model_name}/imu</topic>
+      <gz_frame_id>${prefix}imu_link</gz_frame_id>
+      <imu>
+        <angular_velocity>
+          <x>
+            <noise type="gaussian">
+              <mean>0.0</mean>
+              <stddev>2e-4</stddev>
+              <bias_mean>0.0000075</bias_mean>
+              <bias_stddev>0.0000008</bias_stddev>
+            </noise>
+          </x>
+          <y>
+            <noise type="gaussian">
+              <mean>0.0</mean>
+              <stddev>2e-4</stddev>
+              <bias_mean>0.0000075</bias_mean>
+              <bias_stddev>0.0000008</bias_stddev>
+            </noise>
+          </y>
+          <z>
+            <noise type="gaussian">
+              <mean>0.0</mean>
+              <stddev>2e-4</stddev>
+              <bias_mean>0.0000075</bias_mean>
+              <bias_stddev>0.0000008</bias_stddev>
+            </noise>
+          </z>
+        </angular_velocity>
+        <linear_acceleration>
+          <x>
+            <noise type="gaussian">
+              <mean>0.0</mean>
+              <stddev>1.7e-2</stddev>
+              <bias_mean>0.1</bias_mean>
+              <bias_stddev>0.001</bias_stddev>
+            </noise>
+          </x>
+          <y>
+            <noise type="gaussian">
+              <mean>0.0</mean>
+              <stddev>1.7e-2</stddev>
+              <bias_mean>0.1</bias_mean>
+              <bias_stddev>0.001</bias_stddev>
+            </noise>
+          </y>
+          <z>
+            <noise type="gaussian">
+              <mean>0.0</mean>
+              <stddev>1.7e-2</stddev>
+              <bias_mean>0.1</bias_mean>
+              <bias_stddev>0.001</bias_stddev>
+            </noise>
+          </z>
+        </linear_acceleration>
+      </imu>
+      <plugin
+        filename="ignition-gazebo-imu-system"
+        name="ignition::gazebo::systems::Imu">
+      </plugin>
+    </sensor>
+  </gazebo>
+  <!-- Drive the base.
+       DiffDrive commands the four wheel joints, so a turn is produced the way a
+       real skid-steer Husky produces one. The alternative, VelocityControl,
+       hard-sets the velocity of base_link only; measured on this repository it
+       tracks linear commands exactly but achieves just 0.045 rad/s of the
+       0.5 rad/s commanded yaw, because the wheel contacts resist a rotation
+       that no wheel is turning to create. Nav2 needs rotate-in-place for
+       RotateToGoal and for its spin recovery, so DiffDrive is the default.
+       Set drive_plugin:=velocity_control to compare. -->
+  <xacro:if value="${drive_plugin == 'diff_drive'}">
+    <gazebo>
+      <plugin
+        filename="ignition-gazebo-diff-drive-system"
+        name="ignition::gazebo::systems::DiffDrive">
+        <left_joint>${prefix}front_left_wheel_joint</left_joint>
+        <left_joint>${prefix}rear_left_wheel_joint</left_joint>
+        <right_joint>${prefix}front_right_wheel_joint</right_joint>
+        <right_joint>${prefix}rear_right_wheel_joint</right_joint>
+        <!-- A skid-steer's effective track is wider than its geometric track,
+             because turning drags the tyres sideways. Calibrated against the
+             measured yaw rate in test/movement_test.py; the geometric value is
+             the starting point. -->
+        <wheel_separation>$(arg effective_wheel_separation)</wheel_separation>
+        <wheel_radius>${wheel_radius}</wheel_radius>
+        <topic>model/${gz_model_name}/cmd_vel</topic>
+        <!-- DiffDrive also offers odometry, but this model keeps
+             OdometryPublisher (below) as the single odometry source. Point
+             DiffDrive's own output at unused topics so the two plugins never
+             publish to the same place. -->
+        <odom_topic>model/${gz_model_name}/diff_drive/odometry</odom_topic>
+        <tf_topic>model/${gz_model_name}/diff_drive/tf</tf_topic>
+        <frame_id>${prefix}odom</frame_id>
+        <child_frame_id>${prefix}base_link</child_frame_id>
+        <odom_publish_frequency>1</odom_publish_frequency>
+      </plugin>
+    </gazebo>
+  </xacro:if>
+  <xacro:if value="${drive_plugin == 'velocity_control'}">
+    <gazebo>
+      <plugin
+        filename="ignition-gazebo-velocity-control-system"
+        name="ignition::gazebo::systems::VelocityControl">
+        <topic>model/${gz_model_name}/cmd_vel</topic>
+      </plugin>
+    </gazebo>
+  </xacro:if>
+  <!-- Odometry. Differentiates the simulated pose rather than integrating wheel
+       encoders, so it does not accumulate the slip error that skid-steering
+       creates. The EKF fuses it with the IMU to publish odom->base_link. -->
+  <gazebo>
+    <plugin
+      filename="ignition-gazebo-odometry-publisher-system"
+      name="ignition::gazebo::systems::OdometryPublisher">
+      <topic>model/${gz_model_name}/odometry</topic>
+      <odom_publish_frequency>20</odom_publish_frequency>
+      <odom_frame>${prefix}odom</odom_frame>
+      <robot_base_frame>${prefix}base_link</robot_base_frame>
+    </plugin>
+  </gazebo>
+  <gazebo>
+    <plugin
+      filename="ignition-gazebo-joint-state-publisher-system"
+      name="ignition::gazebo::systems::JointStatePublisher">
+      <topic>model/${gz_model_name}/joint_states</topic>
+    </plugin>
+  </gazebo>
+  <gazebo reference="${prefix}base_scan">
+    <sensor type="gpu_lidar" name="lidar">
+      <pose relative_to='${prefix}base_scan'>0 0 0 0 0 0</pose>
+      <visualize>$(arg laser_visual)</visualize>
+      <topic>model/${gz_model_name}/scan</topic>
+      <update_rate>$(arg lidar_update_rate)</update_rate>
+      <gz_frame_id>${prefix}base_scan</gz_frame_id>
+      <ray>
+        <scan>
+          <horizontal>
+            <samples>$(arg lidar_samples)</samples>
+            <resolution>1</resolution>
+            <min_angle>0.0</min_angle>
+            <max_angle>6.28319</max_angle>
+          </horizontal>
+        </scan>
+        <range>
+          <min>0.2</min>
+          <max>40</max>
+          <resolution>0.015</resolution>
+        </range>
+        <noise>
+          <type>gaussian</type>
+          <mean>0.0</mean>
+          <stddev>0.01</stddev>
+        </noise>
+      </ray>
+      <always_on>true</always_on>
+    </sensor>
+  </gazebo>
+  <xacro:if value="${enable_camera}">
+  <gazebo reference="${prefix}camera_link">
+    <sensor name="rgbd_camera" type="rgbd_camera">
+      <camera>
+        <horizontal_fov>2.0944</horizontal_fov>
+        <image>
+          <width>$(arg camera_width)</width>
+          <height>$(arg camera_height)</height>
+        </image>
+        <clip>
+          <near>0.1</near>
+          <far>40</far>
+        </clip>
+        <!-- depth_camera near/far clip seems to be ignored for some reason -->
+        <!--    We're using Ignition Gazebo Fortress, which uses sdf format 1.9: http://sdformat.org/tutorials?tut=roadmap -->
+        <!--    This takes the depth_camera parameter with near / far clip http://sdformat.org/spec?ver=1.4&elem=sensor  -->
+        <!-- We also use ign sensors v6 ( run ls | grep libignition-sensors in /usr/lib/x86_64-linux-gnu)-->
+        <!-- Looking at the source code, the sdf sets HasDepthCamera() and corresponding HasDepthNearClip() & HasDepthFarClip() which are used in RgbdCameraSensor.cc, so this should work? -->
+        <!--    SDF description of Camera: https://github.com/gazebosim/sdformat/blob/sdf9/src/Camera.cc#L598-->
+        <!--    Camera sensor source code: https://github.com/gazebosim/gz-sensors/blob/ign-sensors6/src/RgbdCameraSensor.cc#L311  -->
+        <depth_camera>
+          <clip>
+            <near>0.4</near>
+            <far>10</far>
+          </clip>
+        </depth_camera>
+      </camera>
+      <always_on>1</always_on>
+      <update_rate>$(arg camera_update_rate)</update_rate>
+      <visualize>$(arg camera_visual)</visualize>
+      <topic>/model/${gz_model_name}/camera</topic>
+      <gz_frame_id>${prefix}camera_link</gz_frame_id>
+    </sensor>
+  </gazebo>
+  </xacro:if>
+  <!-- B.E.E.R. thermal sensor added: beer_thermal_camera -->
+  <gazebo reference="${prefix}camera_link">
+    <!-- B.E.E.R. thermal fire-detection camera -->
+    <sensor name="beer_thermal_camera" type="thermal">
+      <pose>0.45 0 0.45 0 0 0</pose>
+      <camera>
+        <horizontal_fov>1.047</horizontal_fov>
+        <image>
+          <width>320</width>
+          <height>240</height>
+          <format>L16</format>
+        </image>
+        <clip>
+          <near>0.1</near>
+          <far>20.0</far>
+        </clip>
+      </camera>
+      <always_on>true</always_on>
+      <update_rate>10</update_rate>
+      <visualize>true</visualize>
+      <!-- Publish to model-level topic; bridge config maps this to /husky1/thermal/image -->
+      <topic>/model/${gz_model_name}/thermal/image</topic>
+      <plugin
+          filename="ignition-gazebo-thermal-sensor-system"
+          name="ignition::gazebo::systems::ThermalSensor">
+        <min_temp>273.15</min_temp>
+        <max_temp>673.15</max_temp>
+        <resolution>0.01</resolution>
+      </plugin>
+    </sensor>
+  </gazebo>
+</robot>

File: install/41068_ignition_bringup/share/41068_ignition_bringup/urdf_husky/husky.urdf.xacro (robot description, xacro)
@@ -1 +1,170 @@
-/home/jordan/G25_RS1/RS1-Gr25/src/41068_ignition_bringup_v1/41068_ignition_bringup/urdf_husky/husky.urdf.xacro
+<?xml version="1.0" ?>
+<robot name="husky" xmlns:xacro="http://ros.org/wiki/xacro">
+  <xacro:arg name="prefix" default=""/>
+  <xacro:property name="prefix" value="$(arg prefix)"/>
+  <xacro:include filename="$(find 41068_ignition_bringup)/urdf_husky/common_properties.urdf.xacro"/>
+  <xacro:include filename="$(find 41068_ignition_bringup)/urdf_husky/husky.gazebo.xacro"/>
+  <xacro:include filename="$(find 41068_ignition_bringup)/urdf_husky/wheel.urdf.xacro"/>
+  <xacro:property name="r200_cam_rgb_px" value="0.005"/>
+  <xacro:property name="r200_cam_rgb_py" value="0.018"/>
+  <xacro:property name="r200_cam_rgb_pz" value="0.013"/>
+  <xacro:property name="r200_cam_depth_offset" value="0.01"/>
+  <link name="${prefix}base_link">
+    <visual>
+      <origin xyz="0 0 0.0" rpy="0 0 0"/>
+      <geometry>
+        <mesh filename="file://$(find 41068_ignition_bringup)/urdf_husky/meshes/base_link.dae"/>
+      </geometry>
+      <material name="black"/>
+    </visual>
+    <visual name="base_link_fixed_joint_lump__front_bumper_link_visual_3">
+      <origin xyz="0.48 0 0.091" rpy="0 0 0"/>
+      <geometry>
+        <mesh filename="file://$(find 41068_ignition_bringup)/urdf_husky/meshes/bumper.dae"/>
+      </geometry>
+      <material name="black"/>
+    </visual>
+    <visual name="base_link_fixed_joint_lump__rear_bumper_link_visual_4">
+      <origin xyz="-0.48 0 0.091" rpy="0 0 3.14159"/>
+      <geometry>
+        <mesh filename="file://$(find 41068_ignition_bringup)/urdf_husky/meshes/bumper.dae"/>
+      </geometry>
+      <material name="black"/>
+    </visual>
+    <visual name="base_link_fixed_joint_lump__top_chassis_link_visual_5">
+      <origin xyz="0 0 0" rpy="0 0 0"/>
+      <geometry>
+        <mesh filename="file://$(find 41068_ignition_bringup)/urdf_husky/meshes/top_chassis.dae"/>
+      </geometry>
+      <material name="orange"/>
+    </visual>
+    <visual name="base_link_fixed_joint_lump__top_plate_link_visual_6">
+      <origin xyz="0.0812 0 0.245" rpy="0 0 0"/>
+      <geometry>
+        <mesh filename="file://$(find 41068_ignition_bringup)/urdf_husky/meshes/top_plate.dae"/>
+      </geometry>
+      <material name="black"/>
+    </visual>
+    <visual name="base_link_fixed_joint_lump__arch_visual_7">
+      <origin xyz="0.0012 0 0.251" rpy="0 0 0"/>
+      <geometry>
+        <mesh filename="file://$(find 41068_ignition_bringup)/urdf_husky/meshes/jpl04_arch_nosensor.stl"/>
+      </geometry>
+      <material name="black"/>
+    </visual>
+    <collision name="base_link_collision">
+      <origin xyz="0 0 0.12" rpy="0 0 0"/>
+      <geometry>
+        <box size="0.9874 0.5709 0.05"/>
+      </geometry>
+    </collision>
+    <collision name="base_link_collision_bottom">
+      <origin xyz="0 0 0.046" rpy="0 0 0"/>
+      <geometry>
+        <box size="0.80 0.5709 0.095"/>
+      </geometry>
+    </collision>
+    <collision name="base_link_collision_1">
+      <origin xyz="0 0 0.185625" rpy="0 0 0"/>
+      <geometry>
+        <box size="0.78992 0.5709 0.12375"/>
+      </geometry>
+    </collision>
+    <collision name="base_link_fixed_joint_lump__top_plate_link_collision_3">
+      <origin xyz="0.0812 0 0.245" rpy="0 0 0"/>
+      <geometry>
+        <mesh filename="file://$(find 41068_ignition_bringup)/urdf_husky/meshes/top_plate.dae"/>
+      </geometry>
+    </collision>
+    <collision name="base_link_fixed_joint_lump__top_plate_link_collision_4">
+      <origin xyz="0.0812 0 0.245" rpy="0 0 0"/>
+      <geometry>
+        <box size="0.32 0.41 0.09"/>
+      </geometry>
+    </collision>
+    <inertial>
+      <origin xyz="0 0 0.062329" rpy="0 0 0"/>
+      <mass value="46.064"/>
+      <inertia ixx="0.615397" ixy="-0.0240585" ixz="-0.120749"
+               iyy="1.75388" iyz="-0.0028322"
+               izz="2.03641" />
+    </inertial>
+  </link>
+  <!-- Wheels -->
+  <xacro:wheel prefix="${prefix}" wheel_id="front_left" x_pos="0.256" y_pos="${wheel_separation/2}"/>
+  <xacro:wheel prefix="${prefix}" wheel_id="front_right" x_pos="0.256" y_pos="-${wheel_separation/2}"/>
+  <xacro:wheel prefix="${prefix}" wheel_id="rear_left" x_pos="-0.256" y_pos="${wheel_separation/2}"/>
+  <xacro:wheel prefix="${prefix}" wheel_id="rear_right" x_pos="-0.256" y_pos="-${wheel_separation/2}"/>
+  <joint name="${prefix}imu_joint" type="fixed">
+    <parent link="${prefix}base_link"/>
+    <child link="${prefix}imu_link"/>
+    <origin xyz="0.0 0 0.068" rpy="0 0 0"/>
+  </joint>
+  <link name="${prefix}imu_link"/>
+  <joint name="${prefix}scan_joint" type="fixed">
+    <parent link="${prefix}base_link"/>
+    <child link="${prefix}base_scan"/>
+    <origin xyz="0 0 0.68" rpy="0 0 0"/>
+  </joint>
+  <link name="${prefix}base_scan">
+    <visual>
+      <origin xyz="0 0 0" rpy="0 0 0"/>
+      <geometry>
+        <cylinder length="0.04" radius="0.09"/>
+      </geometry>
+      <material name="dark"/>
+    </visual>
+    <inertial>
+      <mass value="0" />
+      <origin xyz="0 0 0" />
+      <inertia ixx="0.001" ixy="0.0" ixz="0.0"
+               iyy="0.001" iyz="0.0"
+               izz="0.001" />
+    </inertial>
+  </link>
+  <joint name="${prefix}camera_joint" type="fixed">
+    <origin xyz="0.45 0.0 0.25" rpy="0 0 0"/> <!-- 0.5 0.0 0.9 -->
+    <parent link="${prefix}base_link"/>
+    <child link="${prefix}camera_link"/>
+  </joint>
+  <link name="${prefix}camera_link">
+    <visual>
+     <origin xyz="0 0 0" rpy="0 0 0"/>
+      <geometry>
+        <box size="0.02 0.08 0.05"/>
+      </geometry>
+      <material name="dark"/>
+    </visual>
+    <visual>
+     <origin xyz="0.015 0 0" rpy="0 1.57 0"/>
+      <geometry>
+        <cylinder length="0.03" radius="0.02"/>
+      </geometry>
+      <material name="dark"/>
+    </visual>
+  </link>
+  <joint name="${prefix}camera_rgb_joint" type="fixed">
+    <origin xyz="${r200_cam_rgb_px} ${r200_cam_rgb_py} ${r200_cam_rgb_pz}" rpy="0 0 0"/>
+    <parent link="${prefix}camera_link"/>
+    <child link="${prefix}camera_rgb_frame"/>
+  </joint>
+  <link name="${prefix}camera_rgb_frame"/>
+  <joint name="${prefix}camera_rgb_optical_joint" type="fixed">
+    <origin xyz="0 0 0" rpy="-1.57 0 -1.57"/>
+    <parent link="${prefix}camera_rgb_frame"/>
+    <child link="${prefix}camera_rgb_optical_frame"/>
+  </joint>
+  <link name="${prefix}camera_rgb_optical_frame"/>
+  <joint name="${prefix}camera_depth_joint" type="fixed">
+    <origin xyz="${r200_cam_rgb_px} ${r200_cam_rgb_py + r200_cam_depth_offset} ${r200_cam_rgb_pz}" rpy="0 0 0"/>
+    <parent link="${prefix}camera_link"/>
+    <child link="${prefix}camera_depth_frame"/>
+  </joint>
+  <link name="${prefix}camera_depth_frame"/>
+  <joint name="${prefix}camera_depth_optical_joint" type="fixed">
+    <origin xyz="0 0 0" rpy="-1.57 0 -1.57"/>
+    <parent link="${prefix}camera_depth_frame"/>
+    <child link="${prefix}camera_depth_optical_frame"/>
+  </joint>
+  <link name="${prefix}camera_depth_optical_frame"/>
+</robot>

File: install/41068_ignition_bringup/share/41068_ignition_bringup/urdf_husky/wheel.urdf.xacro (robot description, xacro)
@@ -1 +1,40 @@
-/home/jordan/G25_RS1/RS1-Gr25/src/41068_ignition_bringup_v1/41068_ignition_bringup/urdf_husky/wheel.urdf.xacro
+<?xml version="1.0"?>
+<robot xmlns:xacro="http://www.ros.org/wiki/xacro" name="wheel">
+  <!-- Properties -->
+  <xacro:property name="wheel_separation" value="0.5708"/>
+  <xacro:property name="wheel_radius" value="0.1651"/>
+  <xacro:macro name="wheel" params="prefix wheel_id x_pos y_pos">
+    <link name="${prefix}${wheel_id}_wheel_link">
+      <visual>
+        <origin xyz="0 0 0" rpy="0 0 0"/>
+        <geometry>
+          <mesh filename="file://$(find 41068_ignition_bringup)/urdf_husky/meshes/wheel.dae"/>
+        </geometry>
+        <material name="dark"/>
+      </visual>
+      <collision>
+        <origin xyz="0 0 0" rpy="1.5707963267948966 0 0"/>
+        <contact_coefficients mu="0.5" kp="1+e07" kd="1"/>
+        <geometry>
+          <cylinder length="0.1143" radius="${wheel_radius}"/>
+        </geometry>
+      </collision>
+      <inertial>
+        <origin xyz="0 0 0" rpy="0 0 0"/>
+        <mass value="2.637"/>
+        <inertia ixx="0.02467" ixy="0" ixz="0"
+                iyy="0.04411" iyz="0"
+                izz="0.02467" />
+      </inertial>
+    </link>
+    <!-- Add joint to main body -->
+    <joint name="${prefix}${wheel_id}_wheel_joint" type="revolute">
+      <parent link="${prefix}base_link"/>
+      <child link="${prefix}${wheel_id}_wheel_link" />
+      <origin xyz="${x_pos} ${y_pos} 0.03282" rpy="0 0 0"/>
+      <limit lower="-1e+16" upper="1e+16" effort="1e+16" velocity="1e+16"/>
+      <axis xyz="0 1 0"/>
+      <dynamics damping="0.004"/>
+    </joint>
+  </xacro:macro>
+</robot>

File: install/41068_ignition_bringup/share/41068_ignition_bringup/urdf_parrot/common_properties.urdf.xacro (robot description, xacro)
@@ -1 +1,34 @@
-/home/jordan/G25_RS1/RS1-Gr25/src/41068_ignition_bringup_v1/41068_ignition_bringup/urdf_parrot/common_properties.urdf.xacro
+<?xml version="1.0" ?>
+<robot name="xacro_properties" xmlns:xacro="http://ros.org/wiki/xacro">
+  <!-- Init colour -->
+  <material name="black">
+      <color rgba="0.0 0.0 0.0 1.0"/>
+  </material>
+  <material name="dark">
+    <color rgba="0.3 0.3 0.3 1.0"/>
+  </material>
+  <material name="light_black">
+    <color rgba="0.4 0.4 0.4 1.0"/>
+  </material>
+  <material name="blue">
+    <color rgba="0.0 0.0 0.8 1.0"/>
+  </material>
+  <material name="green">
+    <color rgba="0.0 0.8 0.0 1.0"/>
+  </material>
+  <material name="grey">
+    <color rgba="0.5 0.5 0.5 1.0"/>
+  </material>
+  <material name="orange">
+    <color rgba="${255/255} ${108/255} ${10/255} 1.0"/>
+  </material>
+  <material name="brown">
+    <color rgba="${222/255} ${207/255} ${195/255} 1.0"/>
+  </material>
+  <material name="red">
+    <color rgba="0.8 0.0 0.0 1.0"/>
+  </material>
+  <material name="white">
+    <color rgba="1.0 1.0 1.0 1.0"/>
+  </material>
+</robot>
